File: Production/SparkFun_MicroMod_ESP32-Panel.brd (EAGLE design)
At the start: 199.6 x 83.1 mm, 822 parts, among them J1 MICROMOD-2222, J10 MICROMOD-2222, J11 MICROMOD-2222, J12 MICROMOD-2222, J13 MICROMOD-2222, J14 MICROMOD-2222, J15 MICROMOD-2222, J16 MICROMOD-2222, J2 MICROMOD-2222, J3 MICROMOD-2222, J4 MICROMOD-2222, J5 MICROMOD-2222, J6 MICROMOD-2222, J7 MICROMOD-2222, J8 MICROMOD-2222, J9 MICROMOD-2222, Q1 MBT3904DW1T1, Q10 MBT3904DW1T1, Q11 MBT3904DW1T1, Q12 MBT3904DW1T1, Q13 MBT3904DW1T1, Q14 MBT3904DW1T1, Q15 MBT3904DW1T1, Q16 MBT3904DW1T1, Q2 MBT3904DW1T1, Q3 MBT3904DW1T1, Q4 MBT3904DW1T1, Q5 MBT3904DW1T1, Q6 MBT3904DW1T1, Q7 MBT3904DW1T1, Q8 MBT3904DW1T1, Q9 MBT3904DW1T1, U1 W25QXX128MBIT-6X5, U10 ESP32, U11 CP2102N, U12 W25QXX128MBIT-6X5, U13 ESP32, U14 CP2102N, U15 W25QXX128MBIT-6X5, U16 ESP32, U17 CP2102N, U18 W25QXX128MBIT-6X5, U19 ESP32, U2 ESP32, U20 CP2102N, U21 W25QXX128MBIT-6X5, U22 ESP32, U23 CP2102N, U24 W25QXX128MBIT-6X5, U25 ESP32, U26 CP2102N, U27 W25QXX128MBIT-6X5, U28 ESP32, U29 CP2102N, U3 ESP32, U30 W25QXX128MBIT-6X5, U31 ESP32, U32 CP2102N, U33 W25QXX128MBIT-6X5, U34 ESP32, U35 CP2102N, U36 W25QXX128MBIT-6X5, U37 ESP32, U38 CP2102N, U39 W25QXX128MBIT-6X5, U4 CP2102N, U40 ESP32, U41 CP2102N, U42 W25QXX128MBIT-6X5, U43 ESP32, U44 CP2102N, U45 W25QXX128MBIT-6X5, U46 ESP32, U47 CP2102N, U48 W25QXX128MBIT-6X5, U5 CP2102N, U6 W25QXX128MBIT-6X5, U7 ESP32, U8 CP2102N, U9 W25QXX128MBIT-6X5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

Commit message: New panel
Connections:
- removed net 0-!BOOT!/I2C_!INT: J1.11, J1.16, Q2.6, R9.1, U2.23
- removed net 0-!BOOT!/I2C_!INT1: J2.11, J2.16, Q1.6, R13.1, U3.23
- removed net 0-!BOOT!/I2C_!INT10: J11.11, J11.16, Q11.6, R96.1, U31.23
- removed net 0-!BOOT!/I2C_!INT11: J12.11, J12.16, Q12.6, R105.1, U34.23
- removed net 0-!BOOT!/I2C_!INT12: J13.11, J13.16, Q13.6, R114.1, U37.23
- removed net 0-!BOOT!/I2C_!INT13: J14.11, J14.16, Q14.6, R123.1, U40.23
- removed net 0-!BOOT!/I2C_!INT14: J15.11, J15.16, Q15.6, R132.1, U43.23
- removed net 0-!BOOT!/I2C_!INT15: J16.11, J16.16, Q16.6, R141.1, U46.23
- removed net 0-!BOOT!/I2C_!INT2: J3.11, J3.16, Q3.6, R24.1, U7.23
- removed net 0-!BOOT!/I2C_!INT3: J4.11, J4.16, Q4.6, R33.1, U10.23
- removed net 0-!BOOT!/I2C_!INT4: J5.11, J5.16, Q5.6, R42.1, U13.23
- removed net 0-!BOOT!/I2C_!INT5: J6.11, J6.16, Q6.6, R51.1, U16.23
- removed net 0-!BOOT!/I2C_!INT6: J7.11, J7.16, Q7.6, R60.1, U19.23
- removed net 0-!BOOT!/I2C_!INT7: J8.11, J8.16, Q8.6, R69.1, U22.23
- removed net 0-!BOOT!/I2C_!INT8: J9.11, J9.16, Q9.6, R78.1, U25.23
- removed net 0-!BOOT!/I2C_!INT9: J10.11, J10.16, Q10.6, R87.1, U28.23
- removed net 16-G2/RX1/AUD_IN: J1.19, J1.44, J1.54, U2.25
- removed net 16-G2/RX1/AUD_IN1: J2.19, J2.44, J2.54, U3.25
- removed net 16-G2/RX1/AUD_IN10: J11.19, J11.44, J11.54, U31.25
- removed net 16-G2/RX1/AUD_IN11: J12.19, J12.44, J12.54, U34.25
- removed net 16-G2/RX1/AUD_IN12: J13.19, J13.44, J13.54, U37.25
- removed net 16-G2/RX1/AUD_IN13: J14.19, J14.44, J14.54, U40.25
- removed net 16-G2/RX1/AUD_IN14: J15.19, J15.44, J15.54, U43.25
- removed net 16-G2/RX1/AUD_IN15: J16.19, J16.44, J16.54, U46.25
- removed net 16-G2/RX1/AUD_IN2: J3.19, J3.44, J3.54, U7.25
- removed net 16-G2/RX1/AUD_IN3: J4.19, J4.44, J4.54, U10.25
- removed net 16-G2/RX1/AUD_IN4: J5.19, J5.44, J5.54, U13.25
- removed net 16-G2/RX1/AUD_IN5: J6.19, J6.44, J6.54, U16.25
- removed net 16-G2/RX1/AUD_IN6: J7.19, J7.44, J7.54, U19.25
- removed net 16-G2/RX1/AUD_IN7: J8.19, J8.44, J8.54, U22.25
- removed net 16-G2/RX1/AUD_IN8: J9.19, J9.44, J9.54, U25.25
- removed net 16-G2/RX1/AUD_IN9: J10.19, J10.44, J10.54, U28.25
- removed net 17-G3/TX1/AUD_OUT: J1.17, J1.46, J1.56, U2.27
- removed net 17-G3/TX1/AUD_OUT1: J2.17, J2.46, J2.56, U3.27
- removed net 17-G3/TX1/AUD_OUT10: J11.17, J11.46, J11.56, U31.27
- removed net 17-G3/TX1/AUD_OUT11: J12.17, J12.46, J12.56, U34.27
- removed net 17-G3/TX1/AUD_OUT12: J13.17, J13.46, J13.56, U37.27
- removed net 17-G3/TX1/AUD_OUT13: J14.17, J14.46, J14.56, U40.27
- removed net 17-G3/TX1/AUD_OUT14: J15.17, J15.46, J15.56, U43.27
- removed net 17-G3/TX1/AUD_OUT15: J16.17, J16.46, J16.56, U46.27
- removed net 17-G3/TX1/AUD_OUT2: J3.17, J3.46, J3.56, U7.27
- removed net 17-G3/TX1/AUD_OUT3: J4.17, J4.46, J4.56, U10.27
- removed net 17-G3/TX1/AUD_OUT4: J5.17, J5.46, J5.56, U13.27
- removed net 17-G3/TX1/AUD_OUT5: J6.17, J6.46, J6.56, U16.27
- removed net 17-G3/TX1/AUD_OUT6: J7.17, J7.46, J7.56, U19.27
- removed net 17-G3/TX1/AUD_OUT7: J8.17, J8.46, J8.56, U22.27
- removed net 17-G3/TX1/AUD_OUT8: J9.17, J9.46, J9.56, U25.27
- removed net 17-G3/TX1/AUD_OUT9: J10.17, J10.46, J10.56, U28.27
- removed net 25-G4/AUD_LRCLK/SCL1: J1.48, J1.52, J1.53, U2.14
- removed net 25-G4/AUD_LRCLK/SCL10: J10.48, J10.52, J10.53, U28.14
- removed net 25-G4/AUD_LRCLK/SCL11: J11.48, J11.52, J11.53, U31.14
- removed net 25-G4/AUD_LRCLK/SCL12: J12.48, J12.52, J12.53, U34.14
- removed net 25-G4/AUD_LRCLK/SCL13: J13.48, J13.52, J13.53, U37.14
- removed net 25-G4/AUD_LRCLK/SCL14: J14.48, J14.52, J14.53, U40.14
- removed net 25-G4/AUD_LRCLK/SCL15: J15.48, J15.52, J15.53, U43.14
- removed net 25-G4/AUD_LRCLK/SCL16: J16.48, J16.52, J16.53, U46.14
- removed net 25-G4/AUD_LRCLK/SCL2: J2.48, J2.52, J2.53, U3.14
- removed net 25-G4/AUD_LRCLK/SCL3: J3.48, J3.52, J3.53, U7.14
- removed net 25-G4/AUD_LRCLK/SCL4: J4.48, J4.52, J4.53, U10.14
- removed net 25-G4/AUD_LRCLK/SCL5: J5.48, J5.52, J5.53, U13.14
- removed net 25-G4/AUD_LRCLK/SCL6: J6.48, J6.52, J6.53, U16.14
- removed net 25-G4/AUD_LRCLK/SCL7: J7.48, J7.52, J7.53, U19.14
- removed net 25-G4/AUD_LRCLK/SCL8: J8.48, J8.52, J8.53, U22.14
- removed net 25-G4/AUD_LRCLK/SCL9: J9.48, J9.52, J9.53, U25.14
- removed net 26-G5/AUD_BCLK/SDA1: J1.50, J1.51, J1.73, U2.15
- removed net 26-G5/AUD_BCLK/SDA10: J10.50, J10.51, J10.73, U28.15
- removed net 26-G5/AUD_BCLK/SDA11: J11.50, J11.51, J11.73, U31.15
- removed net 26-G5/AUD_BCLK/SDA12: J12.50, J12.51, J12.73, U34.15
- removed net 26-G5/AUD_BCLK/SDA13: J13.50, J13.51, J13.73, U37.15
- removed net 26-G5/AUD_BCLK/SDA14: J14.50, J14.51, J14.73, U40.15
- removed net 26-G5/AUD_BCLK/SDA15: J15.50, J15.51, J15.73, U43.15
- removed net 26-G5/AUD_BCLK/SDA16: J16.50, J16.51, J16.73, U46.15
- removed net 26-G5/AUD_BCLK/SDA2: J2.50, J2.51, J2.73, U3.15
- removed net 26-G5/AUD_BCLK/SDA3: J3.50, J3.51, J3.73, U7.15
- removed net 26-G5/AUD_BCLK/SDA4: J4.50, J4.51, J4.73, U10.15
- removed net 26-G5/AUD_BCLK/SDA5: J5.50, J5.51, J5.73, U13.15
- removed net 26-G5/AUD_BCLK/SDA6: J6.50, J6.51, J6.73, U16.15
- removed net 26-G5/AUD_BCLK/SDA7: J7.50, J7.51, J7.73, U19.15
- removed net 26-G5/AUD_BCLK/SDA8: J8.50, J8.51, J8.73, U22.15
- removed net 26-G5/AUD_BCLK/SDA9: J9.50, J9.51, J9.73, U25.15
- removed net 32-G6/RTC: C9.2, J1.71, U2.12, Y2.P$1
- removed net 32-G6/RTC1: C36.2, J2.71, U3.12, Y4.P$1
- removed net 32-G6/RTC10: C216.2, J11.71, U31.12, Y22.P$1
- removed net 32-G6/RTC11: C236.2, J12.71, U34.12, Y24.P$1
- removed net 32-G6/RTC12: C256.2, J13.71, U37.12, Y26.P$1
- removed net 32-G6/RTC13: C276.2, J14.71, U40.12, Y28.P$1
- removed net 32-G6/RTC14: C296.2, J15.71, U43.12, Y30.P$1
- removed net 32-G6/RTC15: C316.2, J16.71, U46.12, Y32.P$1
- removed net 32-G6/RTC2: C56.2, J3.71, U7.12, Y6.P$1
- removed net 32-G6/RTC3: C76.2, J4.71, U10.12, Y8.P$1
- removed net 32-G6/RTC4: C96.2, J5.71, U13.12, Y10.P$1
- removed net 32-G6/RTC5: C116.2, J6.71, U16.12, Y12.P$1
- removed net 32-G6/RTC6: C136.2, J7.71, U19.12, Y14.P$1
- removed net 32-G6/RTC7: C156.2, J8.71, U22.12, Y16.P$1
- removed net 32-G6/RTC8: C176.2, J9.71, U25.12, Y18.P$1
- removed net 32-G6/RTC9: C196.2, J10.71, U28.12, Y20.P$1
- removed net 33-G7/RTC: C26.2, J1.69, U2.13, Y2.P$2
- removed net 33-G7/RTC1: C31.2, J2.69, U3.13, Y4.P$2
- removed net 33-G7/RTC10: C211.2, J11.69, U31.13, Y22.P$2
- removed net 33-G7/RTC11: C231.2, J12.69, U34.13, Y24.P$2
- removed net 33-G7/RTC12: C251.2, J13.69, U37.13, Y26.P$2
- removed net 33-G7/RTC13: C271.2, J14.69, U40.13, Y28.P$2
- removed net 33-G7/RTC14: C291.2, J15.69, U43.13, Y30.P$2
- removed net 33-G7/RTC15: C311.2, J16.69, U46.13, Y32.P$2
- removed net 33-G7/RTC2: C51.2, J3.69, U7.13, Y6.P$2
- removed net 33-G7/RTC3: C71.2, J4.69, U10.13, Y8.P$2
- removed net 33-G7/RTC4: C91.2, J5.69, U13.13, Y10.P$2
- removed net 33-G7/RTC5: C111.2, J6.69, U16.13, Y12.P$2
- removed net 33-G7/RTC6: C131.2, J7.69, U19.13, Y14.P$2
- removed net 33-G7/RTC7: C151.2, J8.69, U22.13, Y16.P$2
- removed net 33-G7/RTC8: C171.2, J9.69, U25.13, Y18.P$2
- removed net 33-G7/RTC9: C191.2, J10.69, U28.13, Y20.P$2
- removed net 4-SD_DATA1/G0: J1.40, J1.66, U2.24
- removed net 4-SD_DATA1/G1: J2.40, J2.66, U3.24
- removed net 4-SD_DATA1/G10: J11.40, J11.66, U31.24
- removed net 4-SD_DATA1/G11: J12.40, J12.66, U34.24
- removed net 4-SD_DATA1/G12: J13.40, J13.66, U37.24
- removed net 4-SD_DATA1/G13: J14.40, J14.66, U40.24
- removed net 4-SD_DATA1/G14: J15.40, J15.66, U43.24
- removed net 4-SD_DATA1/G15: J16.40, J16.66, U46.24
- removed net 4-SD_DATA1/G2: J3.40, J3.66, U7.24
- removed net 4-SD_DATA1/G3: J4.40, J4.66, U10.24
- removed net 4-SD_DATA1/G4: J5.40, J5.66, U13.24
- removed net 4-SD_DATA1/G5: J6.40, J6.66, U16.24
- removed net 4-SD_DATA1/G6: J7.40, J7.66, U19.24
- removed net 4-SD_DATA1/G7: J8.40, J8.66, U22.24
- removed net 4-SD_DATA1/G8: J9.40, J9.66, U25.24
- removed net 4-SD_DATA1/G9: J10.40, J10.66, U28.24
- new net 0-!BOOT!: J1.11, Q2.6, R9.1, U2.23
- new net 0-!BOOT!1: J2.11, Q1.6, R13.1, U3.23
- new net 0-!BOOT!10: J11.11, Q11.6, R96.1, U31.23
- new net 0-!BOOT!11: J12.11, Q12.6, R105.1, U34.23
- new net 0-!BOOT!12: J13.11, Q13.6, R114.1, U37.23
- new net 0-!BOOT!13: J14.11, Q14.6, R123.1, U40.23
- new net 0-!BOOT!14: J15.11, Q15.6, R132.1, U43.23
- new net 0-!BOOT!15: J16.11, Q16.6, R141.1, U46.23
- new net 0-!BOOT!2: J3.11, Q3.6, R24.1, U7.23
- new net 0-!BOOT!3: J4.11, Q4.6, R33.1, U10.23
- new net 0-!BOOT!4: J5.11, Q5.6, R42.1, U13.23
- new net 0-!BOOT!5: J6.11, Q6.6, R51.1, U16.23
- new net 0-!BOOT!6: J7.11, Q7.6, R60.1, U19.23
- new net 0-!BOOT!7: J8.11, Q8.6, R69.1, U22.23
- new net 0-!BOOT!8: J9.11, Q9.6, R78.1, U25.23
- new net 0-!BOOT!9: J10.11, Q10.6, R87.1, U28.23
- new net 16-G3/RX1/AUD_IN: J1.19, J1.46, J1.54, U2.25
- new net 16-G3/RX1/AUD_IN1: J2.19, J2.46, J2.54, U3.25
- new net 16-G3/RX1/AUD_IN10: J11.19, J11.46, J11.54, U31.25
- new net 16-G3/RX1/AUD_IN11: J12.19, J12.46, J12.54, U34.25
- new net 16-G3/RX1/AUD_IN12: J13.19, J13.46, J13.54, U37.25
- new net 16-G3/RX1/AUD_IN13: J14.19, J14.46, J14.54, U40.25
- new net 16-G3/RX1/AUD_IN14: J15.19, J15.46, J15.54, U43.25
- new net 16-G3/RX1/AUD_IN15: J16.19, J16.46, J16.54, U46.25
- new net 16-G3/RX1/AUD_IN2: J3.19, J3.46, J3.54, U7.25
- new net 16-G3/RX1/AUD_IN3: J4.19, J4.46, J4.54, U10.25
- new net 16-G3/RX1/AUD_IN4: J5.19, J5.46, J5.54, U13.25
- new net 16-G3/RX1/AUD_IN5: J6.19, J6.46, J6.54, U16.25
- new net 16-G3/RX1/AUD_IN6: J7.19, J7.46, J7.54, U19.25
- new net 16-G3/RX1/AUD_IN7: J8.19, J8.46, J8.54, U22.25
- new net 16-G3/RX1/AUD_IN8: J9.19, J9.46, J9.54, U25.25
- new net 16-G3/RX1/AUD_IN9: J10.19, J10.46, J10.54, U28.25
- new net 17-G2/TX1/AUD_OUT: J1.17, J1.44, J1.56, U2.27
- new net 17-G2/TX1/AUD_OUT1: J2.17, J2.44, J2.56, U3.27
- new net 17-G2/TX1/AUD_OUT10: J11.17, J11.44, J11.56, U31.27
- new net 17-G2/TX1/AUD_OUT11: J12.17, J12.44, J12.56, U34.27
- new net 17-G2/TX1/AUD_OUT12: J13.17, J13.44, J13.56, U37.27
- new net 17-G2/TX1/AUD_OUT13: J14.17, J14.44, J14.56, U40.27
- new net 17-G2/TX1/AUD_OUT14: J15.17, J15.44, J15.56, U43.27
- new net 17-G2/TX1/AUD_OUT15: J16.17, J16.44, J16.56, U46.27
- new net 17-G2/TX1/AUD_OUT2: J3.17, J3.44, J3.56, U7.27
- new net 17-G2/TX1/AUD_OUT3: J4.17, J4.44, J4.56, U10.27
- new net 17-G2/TX1/AUD_OUT4: J5.17, J5.44, J5.56, U13.27
- new net 17-G2/TX1/AUD_OUT5: J6.17, J6.44, J6.56, U16.27
- new net 17-G2/TX1/AUD_OUT6: J7.17, J7.44, J7.56, U19.27
- new net 17-G2/TX1/AUD_OUT7: J8.17, J8.44, J8.56, U22.27
- new net 17-G2/TX1/AUD_OUT8: J9.17, J9.44, J9.56, U25.27
- new net 17-G2/TX1/AUD_OUT9: J10.17, J10.44, J10.56, U28.27
- new net 25-G0/AUD_LRCLK/SCL1: J1.40, J1.52, J1.53, U2.14
- new net 25-G0/AUD_LRCLK/SCL10: J10.40, J10.52, J10.53, U28.14
- new net 25-G0/AUD_LRCLK/SCL11: J11.40, J11.52, J11.53, U31.14
- new net 25-G0/AUD_LRCLK/SCL12: J12.40, J12.52, J12.53, U34.14
- new net 25-G0/AUD_LRCLK/SCL13: J13.40, J13.52, J13.53, U37.14
- new net 25-G0/AUD_LRCLK/SCL14: J14.40, J14.52, J14.53, U40.14
- new net 25-G0/AUD_LRCLK/SCL15: J15.40, J15.52, J15.53, U43.14
- new net 25-G0/AUD_LRCLK/SCL16: J16.40, J16.52, J16.53, U46.14
- new net 25-G0/AUD_LRCLK/SCL2: J2.40, J2.52, J2.53, U3.14
- new net 25-G0/AUD_LRCLK/SCL3: J3.40, J3.52, J3.53, U7.14
- new net 25-G0/AUD_LRCLK/SCL4: J4.40, J4.52, J4.53, U10.14
- new net 25-G0/AUD_LRCLK/SCL5: J5.40, J5.52, J5.53, U13.14
- new net 25-G0/AUD_LRCLK/SCL6: J6.40, J6.52, J6.53, U16.14
- new net 25-G0/AUD_LRCLK/SCL7: J7.40, J7.52, J7.53, U19.14
- new net 25-G0/AUD_LRCLK/SCL8: J8.40, J8.52, J8.53, U22.14
- new net 25-G0/AUD_LRCLK/SCL9: J9.40, J9.52, J9.53, U25.14
- new net 26-G1/AUD_BCLK/SDA1: J1.42, J1.50, J1.51, U2.15
- new net 26-G1/AUD_BCLK/SDA10: J10.42, J10.50, J10.51, U28.15
- new net 26-G1/AUD_BCLK/SDA11: J11.42, J11.50, J11.51, U31.15
- new net 26-G1/AUD_BCLK/SDA12: J12.42, J12.50, J12.51, U34.15
- new net 26-G1/AUD_BCLK/SDA13: J13.42, J13.50, J13.51, U37.15
- new net 26-G1/AUD_BCLK/SDA14: J14.42, J14.50, J14.51, U40.15
- new net 26-G1/AUD_BCLK/SDA15: J15.42, J15.50, J15.51, U43.15
- new net 26-G1/AUD_BCLK/SDA16: J16.42, J16.50, J16.51, U46.15
- new net 26-G1/AUD_BCLK/SDA2: J2.42, J2.50, J2.51, U3.15
- new net 26-G1/AUD_BCLK/SDA3: J3.42, J3.50, J3.51, U7.15
- new net 26-G1/AUD_BCLK/SDA4: J4.42, J4.50, J4.51, U10.15
- new net 26-G1/AUD_BCLK/SDA5: J5.42, J5.50, J5.51, U13.15
- new net 26-G1/AUD_BCLK/SDA6: J6.42, J6.50, J6.51, U16.15
- new net 26-G1/AUD_BCLK/SDA7: J7.42, J7.50, J7.51, U19.15
- new net 26-G1/AUD_BCLK/SDA8: J8.42, J8.50, J8.51, U22.15
- new net 26-G1/AUD_BCLK/SDA9: J9.42, J9.50, J9.51, U25.15
- new net 32-G5/RTC: C9.2, J1.73, U2.12, Y2.P$1
- new net 32-G5/RTC1: C36.2, J2.73, U3.12, Y4.P$1
- new net 32-G5/RTC10: C216.2, J11.73, U31.12, Y22.P$1
- new net 32-G5/RTC11: C236.2, J12.73, U34.12, Y24.P$1
- new net 32-G5/RTC12: C256.2, J13.73, U37.12, Y26.P$1
- new net 32-G5/RTC13: C276.2, J14.73, U40.12, Y28.P$1
- new net 32-G5/RTC14: C296.2, J15.73, U43.12, Y30.P$1
- new net 32-G5/RTC15: C316.2, J16.73, U46.12, Y32.P$1
- new net 32-G5/RTC2: C56.2, J3.73, U7.12, Y6.P$1
- new net 32-G5/RTC3: C76.2, J4.73, U10.12, Y8.P$1
- new net 32-G5/RTC4: C96.2, J5.73, U13.12, Y10.P$1
- new net 32-G5/RTC5: C116.2, J6.73, U16.12, Y12.P$1
- new net 32-G5/RTC6: C136.2, J7.73, U19.12, Y14.P$1
- new net 32-G5/RTC7: C156.2, J8.73, U22.12, Y16.P$1
- new net 32-G5/RTC8: C176.2, J9.73, U25.12, Y18.P$1
- new net 32-G5/RTC9: C196.2, J10.73, U28.12, Y20.P$1
- new net 33-G6/RTC: C26.2, J1.71, U2.13, Y2.P$2
- new net 33-G6/RTC1: C31.2, J2.71, U3.13, Y4.P$2
- new net 33-G6/RTC10: C211.2, J11.71, U31.13, Y22.P$2
- new net 33-G6/RTC11: C231.2, J12.71, U34.13, Y24.P$2
- new net 33-G6/RTC12: C251.2, J13.71, U37.13, Y26.P$2
- new net 33-G6/RTC13: C271.2, J14.71, U40.13, Y28.P$2
- new net 33-G6/RTC14: C291.2, J15.71, U43.13, Y30.P$2
- new net 33-G6/RTC15: C311.2, J16.71, U46.13, Y32.P$2
- new net 33-G6/RTC2: C51.2, J3.71, U7.13, Y6.P$2
- new net 33-G6/RTC3: C71.2, J4.71, U10.13, Y8.P$2
- new net 33-G6/RTC4: C91.2, J5.71, U13.13, Y10.P$2
- new net 33-G6/RTC5: C111.2, J6.71, U16.13, Y12.P$2
- new net 33-G6/RTC6: C131.2, J7.71, U19.13, Y14.P$2
- new net 33-G6/RTC7: C151.2, J8.71, U22.13, Y16.P$2
- new net 33-G6/RTC8: C171.2, J9.71, U25.13, Y18.P$2
- new net 33-G6/RTC9: C191.2, J10.71, U28.13, Y20.P$2
- new net 4-SD_DATA1/I2C_!INT: J1.16, J1.66, U2.24
- new net 4-SD_DATA1/I2C_!INT1: J2.16, J2.66, U3.24
- new net 4-SD_DATA1/I2C_!INT10: J11.16, J11.66, U31.24
- new net 4-SD_DATA1/I2C_!INT11: J12.16, J12.66, U34.24
- new net 4-SD_DATA1/I2C_!INT12: J13.16, J13.66, U37.24
- new net 4-SD_DATA1/I2C_!INT13: J14.16, J14.66, U40.24
- new net 4-SD_DATA1/I2C_!INT14: J15.16, J15.66, U43.24
- new net 4-SD_DATA1/I2C_!INT15: J16.16, J16.66, U46.24
- new net 4-SD_DATA1/I2C_!INT2: J3.16, J3.66, U7.24
- new net 4-SD_DATA1/I2C_!INT3: J4.16, J4.66, U10.24
- new net 4-SD_DATA1/I2C_!INT4: J5.16, J5.66, U13.24
- new net 4-SD_DATA1/I2C_!INT5: J6.16, J6.66, U16.24
- new net 4-SD_DATA1/I2C_!INT6: J7.16, J7.66, U19.24
- new net 4-SD_DATA1/I2C_!INT7: J8.16, J8.66, U22.24
- new net 4-SD_DATA1/I2C_!INT8: J9.16, J9.66, U25.24
- new net 4-SD_DATA1/I2C_!INT9: J10.16, J10.66, U28.24
- net 12-SD_DATA2/G1: now also J2.48, J2.68, U3.18; no longer J1.42, J1.68, U2.18
- net 12-SD_DATA2/G10: now also J10.48; no longer J10.42
- net 12-SD_DATA2/G11: now also J11.48; no longer J11.42
- net 12-SD_DATA2/G12: now also J12.48; no longer J12.42
- net 12-SD_DATA2/G13: now also J13.48; no longer J13.42
- net 12-SD_DATA2/G14: now also J14.48; no longer J14.42
- net 12-SD_DATA2/G15: now also J15.48; no longer J15.42
- net 12-SD_DATA2/G16: now also J16.48; no longer J16.42
- net 12-SD_DATA2/G2: now also J3.48, J3.68, U7.18; no longer J2.42, J2.68, U3.18
- net 12-SD_DATA2/G3: now also J4.48, J4.68, U10.18; no longer J3.42, J3.68, U7.18
- net 12-SD_DATA2/G4: now also J1.48, J1.68, U2.18; no longer J4.42, J4.68, U10.18
- net 12-SD_DATA2/G5: now also J5.48; no longer J5.42
- net 12-SD_DATA2/G6: now also J6.48; no longer J6.42
- net 12-SD_DATA2/G7: now also J7.48; no longer J7.42
- net 12-SD_DATA2/G8: now also J8.48; no longer J8.42
- net 12-SD_DATA2/G9: now also J9.48; no longer J9.42
Routing:
- net 0-!BOOT!/I2C_!INT15: track 26.7 -> 0.00 mm, vias 3 -> 0
- net 0-!BOOT!/I2C_!INT12: track 26.7 -> 0.00 mm, vias 3 -> 0
- net 0-!BOOT!/I2C_!INT9: track 26.7 -> 0.00 mm, vias 3 -> 0
- net 0-!BOOT!/I2C_!INT8: track 26.7 -> 0.00 mm, vias 3 -> 0
- net 0-!BOOT!/I2C_!INT5: track 26.7 -> 0.00 mm, vias 3 -> 0
- net 0-!BOOT!/I2C_!INT14: track 26.7 -> 0.00 mm, vias 3 -> 0
- net 0-!BOOT!/I2C_!INT13: track 26.7 -> 0.00 mm, vias 3 -> 0
- net 0-!BOOT!/I2C_!INT11: track 26.7 -> 0.00 mm, vias 3 -> 0
- net 0-!BOOT!/I2C_!INT10: track 26.7 -> 0.00 mm, vias 3 -> 0
- net 0-!BOOT!/I2C_!INT4: track 26.7 -> 0.00 mm, vias 3 -> 0
- net 0-!BOOT!/I2C_!INT3: track 26.7 -> 0.00 mm, vias 3 -> 0
- net 0-!BOOT!/I2C_!INT1: track 26.7 -> 0.00 mm, vias 3 -> 0
- net 0-!BOOT!/I2C_!INT: track 26.7 -> 0.00 mm, vias 3 -> 0
- net 0-!BOOT!/I2C_!INT7: track 26.7 -> 0.00 mm, vias 3 -> 0
- net 0-!BOOT!/I2C_!INT6: track 26.7 -> 0.00 mm, vias 3 -> 0
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
Commit message: v11 Panel
Parts:
- U11, U14, U17, U20, U23, U26, U29, U32, U35, U38, U4, U41, U44, U47, U5, U8: value CP2102N -> CP210X
Connections:
- net FLASH_SD_CLK renamed FLASH_SCK
- net FLASH_SD_CLK1 renamed FLASH_SCK1
- net FLASH_SD_CLK10 renamed FLASH_SCK10
- net FLASH_SD_CLK11 renamed FLASH_SCK11
- net FLASH_SD_CLK12 renamed FLASH_SCK12
- net FLASH_SD_CLK13 renamed FLASH_SCK13
- net FLASH_SD_CLK14 renamed FLASH_SCK14
- net FLASH_SD_CLK15 renamed FLASH_SCK15
- net FLASH_SD_CLK2 renamed FLASH_SCK2
- net FLASH_SD_CLK3 renamed FLASH_SCK3
- net FLASH_SD_CLK4 renamed FLASH_SCK4
- net FLASH_SD_CLK5 renamed FLASH_SCK5
- net FLASH_SD_CLK6 renamed FLASH_SCK6
- net FLASH_SD_CLK7 renamed FLASH_SCK7
- net FLASH_SD_CLK8 renamed FLASH_SCK8
- net FLASH_SD_CLK9 renamed FLASH_SCK9
- net FLASH_SD_CMD renamed FLASH_SCS
- net FLASH_SD_CMD1 renamed FLASH_SCS1
- net FLASH_SD_CMD10 renamed FLASH_SCS10
- net FLASH_SD_CMD11 renamed FLASH_SCS11
- net FLASH_SD_CMD12 renamed FLASH_SCS12
- net FLASH_SD_CMD13 renamed FLASH_SCS13
- net FLASH_SD_CMD14 renamed FLASH_SCS14
- net FLASH_SD_CMD15 renamed FLASH_SCS15
- net FLASH_SD_CMD2 renamed FLASH_SCS2
- net FLASH_SD_CMD3 renamed FLASH_SCS3
- net FLASH_SD_CMD4 renamed FLASH_SCS4
- net FLASH_SD_CMD5 renamed FLASH_SCS5
- net FLASH_SD_CMD6 renamed FLASH_SCS6
- net FLASH_SD_CMD7 renamed FLASH_SCS7
- net FLASH_SD_CMD8 renamed FLASH_SCS8
- net FLASH_SD_CMD9 renamed FLASH_SCS9
- net FLASH_SD_DATA0 renamed FLASH_SDO
- net FLASH_SD_DATA1 renamed FLASH_SDI
- net FLASH_SD_DATA10 renamed FLASH_SDI2
- net FLASH_SD_DATA11 renamed FLASH_SDO2
- net FLASH_SD_DATA12 renamed FLASH_SWP3
- net FLASH_SD_DATA13 renamed FLASH_SHD3
- net FLASH_SD_DATA14 renamed FLASH_SDI3
- net FLASH_SD_DATA15 renamed FLASH_SDO3
- net FLASH_SD_DATA16 renamed FLASH_SWP4
- net FLASH_SD_DATA17 renamed FLASH_SHD4
- net FLASH_SD_DATA18 renamed FLASH_SDI4
- net FLASH_SD_DATA19 renamed FLASH_SDO4
- net FLASH_SD_DATA2 renamed FLASH_SHD
- net FLASH_SD_DATA20 renamed FLASH_SWP5
- net FLASH_SD_DATA21 renamed FLASH_SHD5
- net FLASH_SD_DATA22 renamed FLASH_SDI5
- net FLASH_SD_DATA23 renamed FLASH_SDO5
- net FLASH_SD_DATA24 renamed FLASH_SWP6
- net FLASH_SD_DATA25 renamed FLASH_SHD6
- net FLASH_SD_DATA26 renamed FLASH_SDI6
- net FLASH_SD_DATA27 renamed FLASH_SDO6
- net FLASH_SD_DATA28 renamed FLASH_SWP7
- net FLASH_SD_DATA29 renamed FLASH_SHD7
- net FLASH_SD_DATA3 renamed FLASH_SWP
- net FLASH_SD_DATA30 renamed FLASH_SDI7
- net FLASH_SD_DATA31 renamed FLASH_SDO7
- net FLASH_SD_DATA32 renamed FLASH_SWP8
- net FLASH_SD_DATA33 renamed FLASH_SHD8
- net FLASH_SD_DATA34 renamed FLASH_SDI8
- net FLASH_SD_DATA35 renamed FLASH_SDO8
- net FLASH_SD_DATA36 renamed FLASH_SWP9
- net FLASH_SD_DATA37 renamed FLASH_SHD9
- net FLASH_SD_DATA38 renamed FLASH_SDI9
- net FLASH_SD_DATA39 renamed FLASH_SDO9
- net FLASH_SD_DATA4 renamed FLASH_SWP1
- net FLASH_SD_DATA40 renamed FLASH_SWP10
- net FLASH_SD_DATA41 renamed FLASH_SHD10
- net FLASH_SD_DATA42 renamed FLASH_SDI10
- net FLASH_SD_DATA43 renamed FLASH_SDO10
- net FLASH_SD_DATA44 renamed FLASH_SWP11
- net FLASH_SD_DATA45 renamed FLASH_SHD11
- net FLASH_SD_DATA46 renamed FLASH_SDI11
- net FLASH_SD_DATA47 renamed FLASH_SDO11
- net FLASH_SD_DATA48 renamed FLASH_SWP12
- net FLASH_SD_DATA49 renamed FLASH_SHD12
- net FLASH_SD_DATA5 renamed FLASH_SHD1
- net FLASH_SD_DATA50 renamed FLASH_SDI12
- net FLASH_SD_DATA51 renamed FLASH_SDO12
- net FLASH_SD_DATA52 renamed FLASH_SWP13
- net FLASH_SD_DATA53 renamed FLASH_SHD13
- net FLASH_SD_DATA54 renamed FLASH_SDI13
- net FLASH_SD_DATA55 renamed FLASH_SDO13
- net FLASH_SD_DATA56 renamed FLASH_SWP14
- net FLASH_SD_DATA57 renamed FLASH_SHD14
- net FLASH_SD_DATA58 renamed FLASH_SDI14
- net FLASH_SD_DATA59 renamed FLASH_SDO14
- net FLASH_SD_DATA6 renamed FLASH_SDI1
- net FLASH_SD_DATA60 renamed FLASH_SWP15
- net FLASH_SD_DATA61 renamed FLASH_SHD15
- net FLASH_SD_DATA62 renamed FLASH_SDI15
- net FLASH_SD_DATA63 renamed FLASH_SDO15
- net FLASH_SD_DATA7 renamed FLASH_SDO1
- net FLASH_SD_DATA8 renamed FLASH_SWP2
- net FLASH_SD_DATA9 renamed FLASH_SHD2
- removed net 12-SD_DATA2/G1: J2.48, J2.68, U3.18
- removed net 12-SD_DATA2/G10: J10.48, J10.68, U28.18
- removed net 12-SD_DATA2/G11: J11.48, J11.68, U31.18
- removed net 12-SD_DATA2/G12: J12.48, J12.68, U34.18
- removed net 12-SD_DATA2/G13: J13.48, J13.68, U37.18
- removed net 12-SD_DATA2/G14: J14.48, J14.68, U40.18
- removed net 12-SD_DATA2/G15: J15.48, J15.68, U43.18
- removed net 12-SD_DATA2/G16: J16.48, J16.68, U46.18
- removed net 12-SD_DATA2/G2: J3.48, J3.68, U7.18
- removed net 12-SD_DATA2/G3: J4.48, J4.68, U10.18
- removed net 12-SD_DATA2/G4: J1.48, J1.68, U2.18
- removed net 12-SD_DATA2/G5: J5.48, J5.68, U13.18
- removed net 12-SD_DATA2/G6: J6.48, J6.68, U16.18
- removed net 12-SD_DATA2/G7: J7.48, J7.68, U19.18
- removed net 12-SD_DATA2/G8: J8.48, J8.68, U22.18
- removed net 12-SD_DATA2/G9: J9.48, J9.68, U25.18
- removed net 13-SPI_!CS!/SD_DATA1: J2.70, U3.20
- removed net 13-SPI_!CS!/SD_DATA10: J10.70, U28.20
- removed net 13-SPI_!CS!/SD_DATA11: J11.70, U31.20
- removed net 13-SPI_!CS!/SD_DATA12: J12.70, U34.20
- removed net 13-SPI_!CS!/SD_DATA13: J13.70, U37.20
- removed net 13-SPI_!CS!/SD_DATA14: J14.70, U40.20
- removed net 13-SPI_!CS!/SD_DATA15: J15.70, U43.20
- removed net 13-SPI_!CS!/SD_DATA16: J16.70, U46.20
- removed net 13-SPI_!CS!/SD_DATA2: J3.70, U7.20
- removed net 13-SPI_!CS!/SD_DATA3: J1.70, U2.20
- removed net 13-SPI_!CS!/SD_DATA4: J4.70, U10.20
- removed net 13-SPI_!CS!/SD_DATA5: J5.70, U13.20
- removed net 13-SPI_!CS!/SD_DATA6: J6.70, U16.20
- removed net 13-SPI_!CS!/SD_DATA7: J7.70, U19.20
- removed net 13-SPI_!CS!/SD_DATA8: J8.70, U22.20
- removed net 13-SPI_!CS!/SD_DATA9: J9.70, U25.20
- removed net 14-SPI_SCK/SD_CLK: J1.60, U2.17
- removed net 14-SPI_SCK/SD_CLK1: J2.60, U3.17
- removed net 14-SPI_SCK/SD_CLK10: J11.60, U31.17
- removed net 14-SPI_SCK/SD_CLK11: J12.60, U34.17
- removed net 14-SPI_SCK/SD_CLK12: J13.60, U37.17
- removed net 14-SPI_SCK/SD_CLK13: J14.60, U40.17
- removed net 14-SPI_SCK/SD_CLK14: J15.60, U43.17
- removed net 14-SPI_SCK/SD_CLK15: J16.60, U46.17
- removed net 14-SPI_SCK/SD_CLK2: J3.60, U7.17
- removed net 14-SPI_SCK/SD_CLK3: J4.60, U10.17
- removed net 14-SPI_SCK/SD_CLK4: J5.60, U13.17
- removed net 14-SPI_SCK/SD_CLK5: J6.60, U16.17
- removed net 14-SPI_SCK/SD_CLK6: J7.60, U19.17
- removed net 14-SPI_SCK/SD_CLK7: J8.60, U22.17
- removed net 14-SPI_SCK/SD_CLK8: J9.60, U25.17
- removed net 14-SPI_SCK/SD_CLK9: J10.60, U28.17
- removed net 15-SPI_COPI/SD_CMD: J1.62, U2.21
- removed net 15-SPI_COPI/SD_CMD1: J2.62, U3.21
- removed net 15-SPI_COPI/SD_CMD10: J11.62, U31.21
- removed net 15-SPI_COPI/SD_CMD11: J12.62, U34.21
- removed net 15-SPI_COPI/SD_CMD12: J13.62, U37.21
- removed net 15-SPI_COPI/SD_CMD13: J14.62, U40.21
- removed net 15-SPI_COPI/SD_CMD14: J15.62, U43.21
- removed net 15-SPI_COPI/SD_CMD15: J16.62, U46.21
- removed net 15-SPI_COPI/SD_CMD2: J3.62, U7.21
- removed net 15-SPI_COPI/SD_CMD3: J4.62, U10.21
- removed net 15-SPI_COPI/SD_CMD4: J5.62, U13.21
- removed net 15-SPI_COPI/SD_CMD5: J6.62, U16.21
- removed net 15-SPI_COPI/SD_CMD6: J7.62, U19.21
- removed net 15-SPI_COPI/SD_CMD7: J8.62, U22.21
- removed net 15-SPI_COPI/SD_CMD8: J9.62, U25.21
- removed net 15-SPI_COPI/SD_CMD9: J10.62, U28.21
- removed net 16-G3/RX1/AUD_IN: J1.19, J1.46, J1.54, U2.25
- removed net 16-G3/RX1/AUD_IN1: J2.19, J2.46, J2.54, U3.25
- removed net 16-G3/RX1/AUD_IN10: J11.19, J11.46, J11.54, U31.25
- removed net 16-G3/RX1/AUD_IN11: J12.19, J12.46, J12.54, U34.25
- removed net 16-G3/RX1/AUD_IN12: J13.19, J13.46, J13.54, U37.25
- removed net 16-G3/RX1/AUD_IN13: J14.19, J14.46, J14.54, U40.25
- removed net 16-G3/RX1/AUD_IN14: J15.19, J15.46, J15.54, U43.25
- removed net 16-G3/RX1/AUD_IN15: J16.19, J16.46, J16.54, U46.25
- removed net 16-G3/RX1/AUD_IN2: J3.19, J3.46, J3.54, U7.25
- removed net 16-G3/RX1/AUD_IN3: J4.19, J4.46, J4.54, U10.25
- removed net 16-G3/RX1/AUD_IN4: J5.19, J5.46, J5.54, U13.25
- removed net 16-G3/RX1/AUD_IN5: J6.19, J6.46, J6.54, U16.25
- removed net 16-G3/RX1/AUD_IN6: J7.19, J7.46, J7.54, U19.25
- removed net 16-G3/RX1/AUD_IN7: J8.19, J8.46, J8.54, U22.25
- removed net 16-G3/RX1/AUD_IN8: J9.19, J9.46, J9.54, U25.25
- removed net 16-G3/RX1/AUD_IN9: J10.19, J10.46, J10.54, U28.25
- removed net 17-G2/TX1/AUD_OUT: J1.17, J1.44, J1.56, U2.27
- removed net 17-G2/TX1/AUD_OUT1: J2.17, J2.44, J2.56, U3.27
- removed net 17-G2/TX1/AUD_OUT10: J11.17, J11.44, J11.56, U31.27
- removed net 17-G2/TX1/AUD_OUT11: J12.17, J12.44, J12.56, U34.27
- removed net 17-G2/TX1/AUD_OUT12: J13.17, J13.44, J13.56, U37.27
- removed net 17-G2/TX1/AUD_OUT13: J14.17, J14.44, J14.56, U40.27
- removed net 17-G2/TX1/AUD_OUT14: J15.17, J15.44, J15.56, U43.27
- removed net 17-G2/TX1/AUD_OUT15: J16.17, J16.44, J16.56, U46.27
- removed net 17-G2/TX1/AUD_OUT2: J3.17, J3.44, J3.56, U7.27
- removed net 17-G2/TX1/AUD_OUT3: J4.17, J4.44, J4.56, U10.27
- removed net 17-G2/TX1/AUD_OUT4: J5.17, J5.44, J5.56, U13.27
- removed net 17-G2/TX1/AUD_OUT5: J6.17, J6.44, J6.56, U16.27
- removed net 17-G2/TX1/AUD_OUT6: J7.17, J7.44, J7.56, U19.27
- removed net 17-G2/TX1/AUD_OUT7: J8.17, J8.44, J8.56, U22.27
- removed net 17-G2/TX1/AUD_OUT8: J9.17, J9.44, J9.56, U25.27
- removed net 17-G2/TX1/AUD_OUT9: J10.17, J10.44, J10.56, U28.27
- removed net 18-PWM0: J1.32, U2.35
- removed net 18-PWM1: J2.32, U3.35
- removed net 18-PWM10: J11.32, U31.35
- removed net 18-PWM11: J12.32, U34.35
- removed net 18-PWM12: J13.32, U37.35
- removed net 18-PWM13: J14.32, U40.35
- removed net 18-PWM14: J15.32, U43.35
- removed net 18-PWM15: J16.32, U46.35
- removed net 18-PWM2: J3.32, U7.35
- removed net 18-PWM3: J4.32, U10.35
- removed net 18-PWM4: J5.32, U13.35
- removed net 18-PWM5: J6.32, U16.35
- removed net 18-PWM6: J7.32, U19.35
- removed net 18-PWM7: J8.32, U22.35
- removed net 18-PWM8: J9.32, U25.35
- removed net 18-PWM9: J10.32, U28.35
- removed net 19-PWM1: J1.47, U2.38
- removed net 19-PWM10: J10.47, U28.38
- removed net 19-PWM11: J11.47, U31.38
- removed net 19-PWM12: J12.47, U34.38
- removed net 19-PWM13: J13.47, U37.38
- removed net 19-PWM14: J14.47, U40.38
- removed net 19-PWM15: J15.47, U43.38
- removed net 19-PWM16: J16.47, U46.38
- removed net 19-PWM2: J2.47, U3.38
- removed net 19-PWM3: J3.47, U7.38
- removed net 19-PWM4: J4.47, U10.38
- removed net 19-PWM5: J5.47, U13.38
- removed net 19-PWM6: J6.47, U16.38
- removed net 19-PWM7: J7.47, U19.38
- removed net 19-PWM8: J8.47, U22.38
- removed net 19-PWM9: J9.47, U25.38
- removed net 2-SPI_CIPO/SD_DATA0: J1.64, U2.22
- removed net 2-SPI_CIPO/SD_DATA1: J2.64, U3.22
- removed net 2-SPI_CIPO/SD_DATA10: J11.64, U31.22
- removed net 2-SPI_CIPO/SD_DATA11: J12.64, U34.22
- removed net 2-SPI_CIPO/SD_DATA12: J13.64, U37.22
- removed net 2-SPI_CIPO/SD_DATA13: J14.64, U40.22
- removed net 2-SPI_CIPO/SD_DATA14: J15.64, U43.22
- removed net 2-SPI_CIPO/SD_DATA15: J16.64, U46.22
- removed net 2-SPI_CIPO/SD_DATA2: J3.64, U7.22
- removed net 2-SPI_CIPO/SD_DATA3: J4.64, U10.22
- removed net 2-SPI_CIPO/SD_DATA4: J5.64, U13.22
- removed net 2-SPI_CIPO/SD_DATA5: J6.64, U16.22
- removed net 2-SPI_CIPO/SD_DATA6: J7.64, U19.22
- removed net 2-SPI_CIPO/SD_DATA7: J8.64, U22.22
- removed net 2-SPI_CIPO/SD_DATA8: J9.64, U25.22
- removed net 2-SPI_CIPO/SD_DATA9: J10.64, U28.22
- removed net 23-D0: J1.10, U2.36
- removed net 23-D1: J2.10, U3.36
- removed net 23-D10: J11.10, U31.36
- removed net 23-D11: J12.10, U34.36
- removed net 23-D12: J13.10, U37.36
- removed net 23-D13: J14.10, U40.36
- removed net 23-D14: J15.10, U43.36
- removed net 23-D15: J16.10, U46.36
- removed net 23-D2: J3.10, U7.36
- removed net 23-D3: J4.10, U10.36
- removed net 23-D4: J5.10, U13.36
- removed net 23-D5: J6.10, U16.36
- removed net 23-D6: J7.10, U19.36
- removed net 23-D7: J8.10, U22.36
- removed net 23-D8: J9.10, U25.36
- removed net 23-D9: J10.10, U28.36
- removed net 25-G0/AUD_LRCLK/SCL1: J1.40, J1.52, J1.53, U2.14
- removed net 25-G0/AUD_LRCLK/SCL10: J10.40, J10.52, J10.53, U28.14
- removed net 25-G0/AUD_LRCLK/SCL11: J11.40, J11.52, J11.53, U31.14
- removed net 25-G0/AUD_LRCLK/SCL12: J12.40, J12.52, J12.53, U34.14
- removed net 25-G0/AUD_LRCLK/SCL13: J13.40, J13.52, J13.53, U37.14
- removed net 25-G0/AUD_LRCLK/SCL14: J14.40, J14.52, J14.53, U40.14
- removed net 25-G0/AUD_LRCLK/SCL15: J15.40, J15.52, J15.53, U43.14
- removed net 25-G0/AUD_LRCLK/SCL16: J16.40, J16.52, J16.53, U46.14
- removed net 25-G0/AUD_LRCLK/SCL2: J2.40, J2.52, J2.53, U3.14
- removed net 25-G0/AUD_LRCLK/SCL3: J3.40, J3.52, J3.53, U7.14
- removed net 25-G0/AUD_LRCLK/SCL4: J4.40, J4.52, J4.53, U10.14
- removed net 25-G0/AUD_LRCLK/SCL5: J5.40, J5.52, J5.53, U13.14
- removed net 25-G0/AUD_LRCLK/SCL6: J6.40, J6.52, J6.53, U16.14
- removed net 25-G0/AUD_LRCLK/SCL7: J7.40, J7.52, J7.53, U19.14
- removed net 25-G0/AUD_LRCLK/SCL8: J8.40, J8.52, J8.53, U22.14
- removed net 25-G0/AUD_LRCLK/SCL9: J9.40, J9.52, J9.53, U25.14
- removed net 26-G1/AUD_BCLK/SDA1: J1.42, J1.50, J1.51, U2.15
- removed net 26-G1/AUD_BCLK/SDA10: J10.42, J10.50, J10.51, U28.15
- removed net 26-G1/AUD_BCLK/SDA11: J11.42, J11.50, J11.51, U31.15
- removed net 26-G1/AUD_BCLK/SDA12: J12.42, J12.50, J12.51, U34.15
- removed net 26-G1/AUD_BCLK/SDA13: J13.42, J13.50, J13.51, U37.15
- removed net 26-G1/AUD_BCLK/SDA14: J14.42, J14.50, J14.51, U40.15
- removed net 26-G1/AUD_BCLK/SDA15: J15.42, J15.50, J15.51, U43.15
- removed net 26-G1/AUD_BCLK/SDA16: J16.42, J16.50, J16.51, U46.15
- removed net 26-G1/AUD_BCLK/SDA2: J2.42, J2.50, J2.51, U3.15
- removed net 26-G1/AUD_BCLK/SDA3: J3.42, J3.50, J3.51, U7.15
- removed net 26-G1/AUD_BCLK/SDA4: J4.42, J4.50, J4.51, U10.15
- removed net 26-G1/AUD_BCLK/SDA5: J5.42, J5.50, J5.51, U13.15
- removed net 26-G1/AUD_BCLK/SDA6: J6.42, J6.50, J6.51, U16.15
- removed net 26-G1/AUD_BCLK/SDA7: J7.42, J7.50, J7.51, U19.15
- removed net 26-G1/AUD_BCLK/SDA8: J8.42, J8.50, J8.51, U22.15
- removed net 26-G1/AUD_BCLK/SDA9: J9.42, J9.50, J9.51, U25.15
- removed net 4-SD_DATA1/I2C_!INT: J1.16, J1.66, U2.24
- removed net 4-SD_DATA1/I2C_!INT1: J2.16, J2.66, U3.24
- removed net 4-SD_DATA1/I2C_!INT10: J11.16, J11.66, U31.24
- removed net 4-SD_DATA1/I2C_!INT11: J12.16, J12.66, U34.24
- removed net 4-SD_DATA1/I2C_!INT12: J13.16, J13.66, U37.24
- removed net 4-SD_DATA1/I2C_!INT13: J14.16, J14.66, U40.24
- removed net 4-SD_DATA1/I2C_!INT14: J15.16, J15.66, U43.24
- removed net 4-SD_DATA1/I2C_!INT15: J16.16, J16.66, U46.24
- removed net 4-SD_DATA1/I2C_!INT2: J3.16, J3.66, U7.24
- removed net 4-SD_DATA1/I2C_!INT3: J4.16, J4.66, U10.24
- removed net 4-SD_DATA1/I2C_!INT4: J5.16, J5.66, U13.24
- removed net 4-SD_DATA1/I2C_!INT5: J6.16, J6.66, U16.24
- removed net 4-SD_DATA1/I2C_!INT6: J7.16, J7.66, U19.24
- removed net 4-SD_DATA1/I2C_!INT7: J8.16, J8.66, U22.24
- removed net 4-SD_DATA1/I2C_!INT8: J9.16, J9.66, U25.24
- removed net 4-SD_DATA1/I2C_!INT9: J10.16, J10.66, U28.24
- removed net 5-STAT_LED: D4.A, U2.34
- removed net 5-STAT_LED1: D1.A, U3.34
- removed net 5-STAT_LED10: D11.A, U31.34
- removed net 5-STAT_LED11: D12.A, U34.34
- removed net 5-STAT_LED12: D13.A, U37.34
- removed net 5-STAT_LED13: D14.A, U40.34
- removed net 5-STAT_LED14: D15.A, U43.34
- removed net 5-STAT_LED15: D16.A, U46.34
- removed net 5-STAT_LED2: D2.A, U7.34
- removed net 5-STAT_LED3: D3.A, U10.34
- removed net 5-STAT_LED4: D5.A, U13.34
- removed net 5-STAT_LED5: D6.A, U16.34
- removed net 5-STAT_LED6: D7.A, U19.34
- removed net 5-STAT_LED7: D8.A, U22.34
- removed net 5-STAT_LED8: D9.A, U25.34
- removed net 5-STAT_LED9: D10.A, U28.34
- new net 12-PWM1: J1.47, U2.18
- new net 12-PWM10: J10.47, U28.18
- new net 12-PWM11: J11.47, U31.18
- new net 12-PWM12: J12.47, U34.18
- new net 12-PWM13: J13.47, U37.18
- new net 12-PWM14: J14.47, U40.18
- new net 12-PWM15: J15.47, U43.18
- new net 12-PWM16: J16.47, U46.18
- new net 12-PWM2: J2.47, U3.18
- new net 12-PWM3: J3.47, U7.18
- new net 12-PWM4: J4.47, U10.18
- new net 12-PWM5: J5.47, U13.18
- new net 12-PWM6: J6.47, U16.18
- new net 12-PWM7: J7.47, U19.18
- new net 12-PWM8: J8.47, U22.18
- new net 12-PWM9: J9.47, U25.18
- new net 13-PWM0: J1.32, U2.20
- new net 13-PWM1: J2.32, U3.20
- new net 13-PWM10: J11.32, U31.20
- new net 13-PWM11: J12.32, U34.20
- new net 13-PWM12: J13.32, U37.20
- new net 13-PWM13: J14.32, U40.20
- new net 13-PWM14: J15.32, U43.20
- new net 13-PWM15: J16.32, U46.20
- new net 13-PWM2: J3.32, U7.20
- new net 13-PWM3: J4.32, U10.20
- new net 13-PWM4: J5.32, U13.20
- new net 13-PWM5: J6.32, U16.20
- new net 13-PWM6: J7.32, U19.20
- new net 13-PWM7: J8.32, U22.20
- new net 13-PWM8: J9.32, U25.20
- new net 13-PWM9: J10.32, U28.20
- new net 14-D0: J1.10, U2.17
- new net 14-D1: J2.10, U3.17
- new net 14-D10: J11.10, U31.17
- new net 14-D11: J12.10, U34.17
- new net 14-D12: J13.10, U37.17
- new net 14-D13: J14.10, U40.17
- new net 14-D14: J15.10, U43.17
- new net 14-D15: J16.10, U46.17
- new net 14-D2: J3.10, U7.17
- new net 14-D3: J4.10, U10.17
- new net 14-D4: J5.10, U13.17
- new net 14-D5: J6.10, U16.17
- new net 14-D6: J7.10, U19.17
- new net 14-D7: J8.10, U22.17
- new net 14-D8: J9.10, U25.17
- new net 14-D9: J10.10, U28.17
- new net 15-G0: J1.40, U2.21
- new net 15-G1: J2.40, U3.21
- new net 15-G10: J11.40, U31.21
- new net 15-G11: J12.40, U34.21
- new net 15-G12: J13.40, U37.21
- new net 15-G13: J14.40, U40.21
- new net 15-G14: J15.40, U43.21
- new net 15-G15: J16.40, U46.21
- new net 15-G2: J3.40, U7.21
- new net 15-G3: J4.40, U10.21
- new net 15-G4: J5.40, U13.21
- new net 15-G5: J6.40, U16.21
- new net 15-G6: J7.40, U19.21
- new net 15-G7: J8.40, U22.21
- new net 15-G8: J9.40, U25.21
- new net 15-G9: J10.40, U28.21
- new net 16-G4/RX1/AUD_IN: J1.19, J1.48, J1.54, U2.25
- new net 16-G4/RX1/AUD_IN1: J2.19, J2.48, J2.54, U3.25
- new net 16-G4/RX1/AUD_IN10: J11.19, J11.48, J11.54, U31.25
- new net 16-G4/RX1/AUD_IN11: J12.19, J12.48, J12.54, U34.25
- new net 16-G4/RX1/AUD_IN12: J13.19, J13.48, J13.54, U37.25
- new net 16-G4/RX1/AUD_IN13: J14.19, J14.48, J14.54, U40.25
- new net 16-G4/RX1/AUD_IN14: J15.19, J15.48, J15.54, U43.25
- new net 16-G4/RX1/AUD_IN15: J16.19, J16.48, J16.54, U46.25
- new net 16-G4/RX1/AUD_IN2: J3.19, J3.48, J3.54, U7.25
- new net 16-G4/RX1/AUD_IN3: J4.19, J4.48, J4.54, U10.25
- new net 16-G4/RX1/AUD_IN4: J5.19, J5.48, J5.54, U13.25
- new net 16-G4/RX1/AUD_IN5: J6.19, J6.48, J6.54, U16.25
- new net 16-G4/RX1/AUD_IN6: J7.19, J7.48, J7.54, U19.25
- new net 16-G4/RX1/AUD_IN7: J8.19, J8.48, J8.54, U22.25
- new net 16-G4/RX1/AUD_IN8: J9.19, J9.48, J9.54, U25.25
- new net 16-G4/RX1/AUD_IN9: J10.19, J10.48, J10.54, U28.25
- new net 17-G3/TX1/AUD_OUT: J1.17, J1.46, J1.56, U2.27
- new net 17-G3/TX1/AUD_OUT1: J2.17, J2.46, J2.56, U3.27
- new net 17-G3/TX1/AUD_OUT10: J11.17, J11.46, J11.56, U31.27
- new net 17-G3/TX1/AUD_OUT11: J12.17, J12.46, J12.56, U34.27
- new net 17-G3/TX1/AUD_OUT12: J13.17, J13.46, J13.56, U37.27
- new net 17-G3/TX1/AUD_OUT13: J14.17, J14.46, J14.56, U40.27
- new net 17-G3/TX1/AUD_OUT14: J15.17, J15.46, J15.56, U43.27
- new net 17-G3/TX1/AUD_OUT15: J16.17, J16.46, J16.56, U46.27
- new net 17-G3/TX1/AUD_OUT2: J3.17, J3.46, J3.56, U7.27
- new net 17-G3/TX1/AUD_OUT3: J4.17, J4.46, J4.56, U10.27
- new net 17-G3/TX1/AUD_OUT4: J5.17, J5.46, J5.56, U13.27
- new net 17-G3/TX1/AUD_OUT5: J6.17, J6.46, J6.56, U16.27
- new net 17-G3/TX1/AUD_OUT6: J7.17, J7.46, J7.56, U19.27
- new net 17-G3/TX1/AUD_OUT7: J8.17, J8.46, J8.56, U22.27
- new net 17-G3/TX1/AUD_OUT8: J9.17, J9.46, J9.56, U25.27
- new net 17-G3/TX1/AUD_OUT9: J10.17, J10.46, J10.56, U28.27
- new net 18-SCK: J1.57, U2.35
- new net 18-SCK1: J2.57, U3.35
- new net 18-SCK10: J11.57, U31.35
- new net 18-SCK11: J12.57, U34.35
- new net 18-SCK12: J13.57, U37.35
- new net 18-SCK13: J14.57, U40.35
- new net 18-SCK14: J15.57, U43.35
- new net 18-SCK15: J16.57, U46.35
- new net 18-SCK2: J3.57, U7.35
- new net 18-SCK3: J4.57, U10.35
- new net 18-SCK4: J5.57, U13.35
- new net 18-SCK5: J6.57, U16.35
- new net 18-SCK6: J7.57, U19.35
- new net 18-SCK7: J8.57, U22.35
- new net 18-SCK8: J9.57, U25.35
- new net 18-SCK9: J10.57, U28.35
- new net 19-CIPO: J1.61, U2.38
- new net 19-CIPO1: J2.61, U3.38
- new net 19-CIPO10: J11.61, U31.38
- new net 19-CIPO11: J12.61, U34.38
- new net 19-CIPO12: J13.61, U37.38
- new net 19-CIPO13: J14.61, U40.38
- new net 19-CIPO14: J15.61, U43.38
- new net 19-CIPO15: J16.61, U46.38
- new net 19-CIPO2: J3.61, U7.38
- new net 19-CIPO3: J4.61, U10.38
- new net 19-CIPO4: J5.61, U13.38
- new net 19-CIPO5: J6.61, U16.38
- new net 19-CIPO6: J7.61, U19.38
- new net 19-CIPO7: J8.61, U22.38
- new net 19-CIPO8: J9.61, U25.38
- new net 19-CIPO9: J10.61, U28.38
- new net 2-STAT_LED: D4.A, U2.22
- new net 2-STAT_LED1: D1.A, U3.22
- new net 2-STAT_LED10: D11.A, U31.22
- new net 2-STAT_LED11: D12.A, U34.22
- new net 2-STAT_LED12: D13.A, U37.22
- new net 2-STAT_LED13: D14.A, U40.22
- new net 2-STAT_LED14: D15.A, U43.22
- new net 2-STAT_LED15: D16.A, U46.22
- new net 2-STAT_LED2: D2.A, U7.22
- new net 2-STAT_LED3: D3.A, U10.22
- new net 2-STAT_LED4: D5.A, U13.22
- new net 2-STAT_LED5: D6.A, U16.22
- new net 2-STAT_LED6: D7.A, U19.22
- new net 2-STAT_LED7: D8.A, U22.22
- new net 2-STAT_LED8: D9.A, U25.22
- new net 2-STAT_LED9: D10.A, U28.22
- new net 23-COPI: J1.59, U2.36
- new net 23-COPI1: J2.59, U3.36
- new net 23-COPI10: J11.59, U31.36
- new net 23-COPI11: J12.59, U34.36
- new net 23-COPI12: J13.59, U37.36
- new net 23-COPI13: J14.59, U40.36
- new net 23-COPI14: J15.59, U43.36
- new net 23-COPI15: J16.59, U46.36
- new net 23-COPI2: J3.59, U7.36
- new net 23-COPI3: J4.59, U10.36
- new net 23-COPI4: J5.59, U13.36
- new net 23-COPI5: J6.59, U16.36
- new net 23-COPI6: J7.59, U19.36
- new net 23-COPI7: J8.59, U22.36
- new net 23-COPI8: J9.59, U25.36
- new net 23-COPI9: J10.59, U28.36
- new net 25-G1/AUD_LRCLK/SCL1: J1.42, J1.52, J1.53, U2.14
- new net 25-G1/AUD_LRCLK/SCL10: J10.42, J10.52, J10.53, U28.14
- new net 25-G1/AUD_LRCLK/SCL11: J11.42, J11.52, J11.53, U31.14
- new net 25-G1/AUD_LRCLK/SCL12: J12.42, J12.52, J12.53, U34.14
- new net 25-G1/AUD_LRCLK/SCL13: J13.42, J13.52, J13.53, U37.14
- new net 25-G1/AUD_LRCLK/SCL14: J14.42, J14.52, J14.53, U40.14
- new net 25-G1/AUD_LRCLK/SCL15: J15.42, J15.52, J15.53, U43.14
- new net 25-G1/AUD_LRCLK/SCL16: J16.42, J16.52, J16.53, U46.14
- new net 25-G1/AUD_LRCLK/SCL2: J2.42, J2.52, J2.53, U3.14
- new net 25-G1/AUD_LRCLK/SCL3: J3.42, J3.52, J3.53, U7.14
- new net 25-G1/AUD_LRCLK/SCL4: J4.42, J4.52, J4.53, U10.14
- new net 25-G1/AUD_LRCLK/SCL5: J5.42, J5.52, J5.53, U13.14
- new net 25-G1/AUD_LRCLK/SCL6: J6.42, J6.52, J6.53, U16.14
- new net 25-G1/AUD_LRCLK/SCL7: J7.42, J7.52, J7.53, U19.14
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Routing:
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Other:
- board text added: "v11"
- board text removed: "v10"
